File: discipline-pcb.kicad_sch (KiCad schematic)
At the start: 161 parts, among them J1 AVR-ISP-6, SW1 KEYSW, SW10 KEYSW, SW11 KEYSW, SW12 KEYSW, SW13 KEYSW, SW14 KEYSW, SW15 KEYSW, SW16 KEYSW, SW17 KEYSW, SW18 KEYSW, SW19 KEYSW, SW2 KEYSW, SW20 KEYSW, SW21 KEYSW, SW22 KEYSW, SW23 KEYSW, SW24 KEYSW, SW25 KEYSW, SW26 KEYSW, SW27 KEYSW, SW28 KEYSW, SW29 KEYSW, SW3 KEYSW, SW30 KEYSW, SW31 KEYSW, SW32 KEYSW, SW33 KEYSW, SW34 KEYSW, SW35 KEYSW, SW36 KEYSW, SW37 KEYSW, SW38 KEYSW, SW39 KEYSW, SW4 KEYSW, SW40 KEYSW, SW41 KEYSW, SW42 KEYSW, SW43 KEYSW, SW44 KEYSW, SW45 KEYSW, SW46 KEYSW, SW47 KEYSW, SW48 KEYSW, SW49 KEYSW, SW5 KEYSW, SW50 KEYSW, SW51 KEYSW, SW52 KEYSW, SW53 KEYSW, SW54 KEYSW, SW55 KEYSW, SW56 KEYSW, SW57 KEYSW, SW58 KEYSW, SW59 KEYSW, SW6 KEYSW, SW60 KEYSW, SW61 KEYSW, SW62 KEYSW, SW63 KEYSW, SW64 KEYSW, SW65 KEYSW, SW66 KEYSW, SW67 KEYSW, SW68 KEYSW, SW7 KEYSW, SW73 KEYSW, SW74 KEYSW, SW8 KEYSW, SW9 KEYSW, U1 ATmega32A-PU, Y1 Crystal

Commit message: use sensible matrix
Parts:
- removed C1, C2: 22p, cftkb:D_DO-35_SOD27_P5.08mm_Horizontal, symbol Device:C_Small
- removed C3: 4.7u, cftkb:D_DO-35_SOD27_P5.08mm_Horizontal, symbol discipline-pcb-rescue:CP1_Small-Device
- removed C4, C5: 0.1u, cftkb:D_DO-35_SOD27_P5.08mm_Horizontal, symbol Device:C_Small
- removed D15, D30, D44, D57, D58, D65, D66, D67: ~, cftkb:D_DO-35_SOD27_P5.08mm_Horizontal, symbol Device:D
- removed D69, D70: 3.6V, cftkb:D_DO-35_SOD27_P5.08mm_Horizontal, symbol Device:D_Zener_Small
- removed J1: AVR-ISP-6, cftkb:AVR_ICSP_3x2, symbol discipline-pcb-rescue:AVR-ISP-6-Connector
- removed R1, R2: 5.1k, cftkb:R_Axial_DIN0204_L3.6mm_D1.6mm_P7.62mm_Horizontal, symbol Device:R_Small
- removed R3, R4: 75R, cftkb:R_Axial_DIN0204_L3.6mm_D1.6mm_P7.62mm_Horizontal, symbol Device:R_Small
- removed R5: 1.5k, cftkb:R_Axial_DIN0204_L3.6mm_D1.6mm_P7.62mm_Horizontal, symbol Device:R_Small
- removed SW15, SW30, SW44, SW57, SW58, SW65, SW66, SW67: KEYSW, cftkb:SW_Cherry_MX1A_1.00u_PCB-NOSCREEN, symbol discipline-pcb-rescue:KEYSW-keyboard_parts
- removed U1: ATmega32A-PU, cftkb:DIP-40_W15.24mm, symbol discipline-pcb-rescue:ATmega32A-PU-MCU_Microchip_ATmega
- removed USB1: USB_C_GCT_USB4085, cftkb:USB_C_GCT_USB4085, symbol discipline-pcb-rescue:USB_C_GCT_USB4085-Type-C
- removed Y1: Crystal, cftkb:Crystal_HC49-4H_Vertical, symbol Device:Crystal
- added D69, D70, D72, D75, D76, D77, D78, D79, D80, D81: ~, cftkb:D_DO-35_SOD27_P5.08mm_Horizontal, symbol Device:D
- added SW69, SW70, SW72, SW75, SW76, SW77, SW78, SW79, SW80, SW81: KEYSW, cftkb:SW_Cherry_MX1A_1.00u_PCB-NOSCREEN, symbol discipline-pcb-rescue:KEYSW-keyboard_parts
Connections:
- net VCC is gone; now on an unnamed net: F1.2
- net GND: now also A1.13 (GND), A1.18 (GND), A1.23 (GND), A1.28 (GND), A1.3 (GND), A1.38 (GND), A1.8 (GND)
- net col0: now also A1.26 (GPIO20)
- net col1: now also A1.25 (GPIO19)
- net col10: now also A1.14 (GPIO10)
- net col11: now also A1.12 (GPIO9)
- net col12: now also A1.11 (GPIO8)
- net col13: now also A1.10 (GPIO7)
- net col14: now also A1.5 (GPIO3), A1.6 (GPIO4), A1.7 (GPIO5), A1.9 (GPIO6), SW69.1, SW70.1, SW72.1, SW75.1, SW76.1, SW77.1, SW78.1, SW79.1, SW80.1, SW81.1
- net col2: now also A1.24 (GPIO18)
- net col3: now also A1.22 (GPIO17)
- net col4: now also A1.21 (GPIO16)
- net col5: now also A1.20 (GPIO15)
- net col6: now also A1.19 (GPIO14)
- net col7: now also A1.17 (GPIO13)
- net col8: now also A1.16 (GPIO12)
- net col9: now also A1.15 (GPIO11)
- net row0: now also A1.34 (GPIO28_ADC2), D69.1 (K), D75.1 (K), D79.1 (K)
- net row1: now also A1.32 (GPIO27_ADC1), D70.1 (K), D76.1 (K), D80.1 (K)
- net row2: now also A1.31 (GPIO26_ADC0)
- net row3: now also A1.29 (GPIO22), D77.1 (K)
- net row4: now also A1.27 (GPIO21), D72.1 (K), D78.1 (K), D81.1 (K)
- new net: D76.2 (A), SW76.2
- new net: D79.2 (A), SW79.2
- new net: D78.2 (A), SW78.2
- new net: D69.2 (A), SW69.2
- new net: D80.2 (A), SW80.2
- new net: D72.2 (A), SW72.2
- new net: D75.2 (A), SW75.2
- new net: D81.2 (A), SW81.2
- new net: D70.2 (A), SW70.2
- no-connect marks 9 -> 2
Other:
- moved on the sheet: A1

Commit message: sort spacings and fix
Parts:
- removed D68: ~, cftkb:D_DO-35_SOD27_P5.08mm_Horizontal, symbol Device:D
- removed SW63, SW64: KEYSW, cftkb:SW_Cherry_MX1A_1.25u_PCBNOSCREEN, symbol discipline-pcb-rescue:KEYSW-keyboard_parts
- removed SW68: KEYSW, cftkb:SW_Cherry_MX1A_1.00u_PCB-NOSCREEN, symbol discipline-pcb-rescue:KEYSW-keyboard_parts
- added D57: ~, cftkb:D_DO-35_SOD27_P5.08mm_Horizontal, symbol Device:D
- added SW57: KEYSW, cftkb:SW_Cherry_MX1A_1.25u_PCBNOSCREEN, symbol discipline-pcb-rescue:KEYSW-keyboard_parts
- SW56: footprint cftkb:SW_Cherry_MX1A_1.75u_PCBNOSCREEN -> cftkb:SW_Cherry_MX1A_2.75u_PCB_NOSCREEN
Connections:
- net col11: now also SW57.1
- net row4: now also D57.1 (K)
- new net: D57.2 (A), SW57.2

Commit message: add stabs, update footprint for cpico
Parts:
- A1: footprint Module:RaspberryPi_Pico_Common_Unspecified -> cftkb:RaspberryPi_CPico
Changed lines of the file:
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@@
 			)
 		)
-		(property "Footprint" "Module:RaspberryPi_Pico_Common_Unspecified"
+		(property "Footprint" "cftkb:RaspberryPi_CPico"
 			(at 264.16 264.16 0)
 			(effects

Commit message: significant improvements to placement
Parts:
- removed D69, D70: ~, cftkb:D_DO-35_SOD27_P5.08mm_Horizontal, symbol Device:D
- removed SW69, SW70: KEYSW, cftkb:SW_Cherry_MX1A_1.00u_PCB-NOSCREEN, symbol discipline-pcb-rescue:KEYSW-keyboard_parts
- renumbered D63 to D73, D64 to D74

Commit message: gross layout looking better
Parts:
- removed BOOT1: BOOT, cftkb:SW_PUSH_6mm, symbol discipline-pcb-rescue:SW_PUSH-keyboard_parts
- removed R7: 10k, cftkb:R_Axial_DIN0204_L3.6mm_D1.6mm_P7.62mm_Horizontal, symbol Device:R_Small
- removed RESET1: RESET, cftkb:SW_PUSH_6mm, symbol discipline-pcb-rescue:SW_PUSH-keyboard_parts
- added D82, D83: ~, cftkb:D_DO-35_SOD27_P5.08mm_Horizontal, symbol Device:D
- added SW82, SW83: KEYSW, cftkb:SW_Cherry_MX1A_1.00u_PCB-NOSCREEN, symbol discipline-pcb-rescue:KEYSW-keyboard_parts
Connections:
- net col14: now also SW82.1, SW83.1
- net row0: now also D82.1 (K)
- net row1: now also D83.1 (K)
- new net: D82.2 (A), SW82.2
- new net: D83.2 (A), SW83.2

Commit message: starting to look like something
Parts:
- removed F1: 500mA, cftkb:polyfuse_5.1mm, symbol Device:Polyfuse_Small
Connections:
- net +5V: now also A1.40 (VBUS)
Changed lines of the file:
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@@
 	(wire
 		(pts
+			(xy 264.16 165.1) (xy 264.16 179.07)
+		)
+		(stroke
+			(width 0)
+			(type default)
+		)
+	)
+	(wire
+		(pts
 			(xy 238.76 232.41) (xy 241.3 232.41)
 		)
@@
 	(wire
 		(pts
-			(xy 264.16 170.18) (xy 264.16 179.07)
-		)
-		(stroke
-			(width 0)
-			(type default)
-		)
-	)
-	(wire
-		(pts
 			(xy 92.71 88.9) (xy 91.44 88.9)
 		)
@@
 					(unit 1)
 				)
-			)
-		)
-	)
-	(symbol
-		(lib_id "Device:Polyfuse_Small")
-		(at 264.16 167.64 0)
-		(unit 1)
-		(exclude_from_sim no)
-		(in_bom yes)
-		(on_board yes)
-		(dnp no)
-		(property "Reference" "F1"
-			(at 265.8872 166.4716 0)
-			(effects
-				(font
-					(size 1.27 1.27)
-				)
-				(justify left)
-			)
-		)
-		(property "Value" "500mA"
-			(at 265.8872 168.783 0)
-			(effects
-				(font
-					(size 1.27 1.27)
-				)
-				(justify left)
-			)
-		)
-		(property "Footprint" "cftkb:polyfuse_5.1mm"
-			(at 265.43 172.72 0)
-			(effects
-				(font
-					(size 1.27 1.27)
-				)
-				(justify left)
-				(hide yes)
-			)
-		)
-		(property "Datasheet" "~"
-			(at 264.16 167.64 0)
-			(effects
-				(font
-					(size 1.27 1.27)
-				)
-				(hide yes)
-			)
-		)
-		(property "Description" ""
-			(at 264.16 167.64 0)
-			(effects
-				(font
-					(size 1.27 1.27)
-				)
-			)
-		)
-		(pin "1"
-		)
-		(pin "2"
-		)
-		(instances
-			(project "discipline-pcb"
-				(path "/92ddd8bc-b115-4355-8708-2687f9ad53cd"
-					(reference "F1")
-					(unit 1)
-				)

Commit message: routing
Connections:
- net at D77.2 (A): now also SW77.2
Changed lines of the file:
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@@
+	(wire
+		(pts
+			(xy 359.41 119.38) (xy 358.14 119.38)
+		)
+		(stroke
+			(width 0)
+			(type default)
+		)
+	)
+	(wire
+		(pts
+			(xy 358.14 119.38) (xy 358.14 120.65)
+		)
+		(stroke
+			(width 0)
+			(type default)
+		)
+	)
 	(wire
 		(pts

Commit message: update nets
Connections:
- net col10: now also SW73.1; no longer SW74.1
- net col11: now also SW74.1; no longer SW57.1
- net col13: now also SW57.1
- net col14: no longer A1.5 (GPIO3), A1.6 (GPIO4), A1.7 (GPIO5), SW75.1, SW76.1, SW77.1, SW78.1, SW79.1, SW80.1, SW81.1
- net col9: no longer SW73.1
- new net col15: A1.7 (GPIO5), SW75.1, SW76.1, SW77.1, SW78.1
- new net col16: A1.6 (GPIO4), SW79.1, SW80.1, SW81.1
Other:
- moved on the sheet: D57, D73, D74, SW57, SW73, SW74
