File: discipline-pcb.kicad_pcb (KiCad board)
At the start: 2 copper layers, 357.2 x 120.3 mm, 150 parts, among them SW1 KEYSW, SW10 KEYSW, SW11 KEYSW, SW12 KEYSW, SW13 KEYSW, SW14 KEYSW, SW16 KEYSW, SW17 KEYSW, SW18 KEYSW, SW19 KEYSW, SW2 KEYSW, SW20 KEYSW, SW21 KEYSW, SW22 KEYSW, SW23 KEYSW, SW24 KEYSW, SW25 KEYSW, SW26 KEYSW, SW27 KEYSW, SW28 KEYSW, SW29 KEYSW, SW3 KEYSW, SW31 KEYSW, SW32 KEYSW, SW33 KEYSW, SW34 KEYSW, SW35 KEYSW, SW36 KEYSW, SW37 KEYSW, SW38 KEYSW, SW39 KEYSW, SW4 KEYSW, SW40 KEYSW, SW41 KEYSW, SW42 KEYSW, SW43 KEYSW, SW45 KEYSW, SW46 KEYSW, SW47 KEYSW, SW48 KEYSW, SW49 KEYSW, SW5 KEYSW, SW50 KEYSW, SW51 KEYSW, SW52 KEYSW, SW53 KEYSW, SW54 KEYSW, SW55 KEYSW, SW56 KEYSW, SW57 KEYSW, SW59 KEYSW, SW6 KEYSW, SW60 KEYSW, SW61 KEYSW, SW62 KEYSW, SW7 KEYSW, SW72 KEYSW, SW73 KEYSW, SW74 KEYSW, SW75 KEYSW, SW76 KEYSW, SW77 KEYSW, SW78 KEYSW, SW79 KEYSW, SW8 KEYSW, SW80 KEYSW, SW81 KEYSW, SW82 KEYSW, SW83 KEYSW, SW9 KEYSW

Commit message: more routing
Parts:
- moved D14 49.8 mm to (330.2, 72.2)
- moved D81 41.9 mm to (288.3, 70.4)
- moved REF** 38.1 mm to (189.4, 64.0)
- moved D57 35.0 mm to (257.9, 65.0)
- moved D74 30.9 mm to (238.8, 65.0)
- moved D73 30.9 mm to (219.8, 65.0)
- moved D12 19.0 mm to (273.1, 72.2)
- moved D13 19.0 mm to (292.1, 72.2)
- moved D11 19.0 mm to (254.1, 72.2)
- moved D10 16.8 mm to (235.0, 72.2)
- moved D27 12.6 mm to (269.3, 70.4)
- moved D26 12.6 mm to (250.3, 70.4)
- moved D43 12.6 mm to (276.9, 65.0)
- moved D25 8.41 mm to (231.2, 70.4)
- moved D54 8.41 mm to (223.6, 66.8)
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Routing:
- net Net-(D57-A): track 0.00 -> 129.4 mm
- net Net-(D74-A): track 0.00 -> 127.5 mm
- net Net-(D73-A): track 0.00 -> 118.0 mm
- net Net-(D56-A): track 0.00 -> 103.5 mm
- net Net-(D55-A): track 0.00 -> 89.2 mm
- net Net-(D54-A): track 0.00 -> 89.2 mm
- net Net-(D43-A): track 0.00 -> 76.3 mm
- net Net-(D29-A): track 0.00 -> 63.6 mm
- net Net-(D40-A): track 0.00 -> 62.8 mm
- net Net-(D42-A): track 0.00 -> 62.8 mm
- net Net-(D41-A): track 0.00 -> 62.8 mm
- net Net-(D28-A): track 0.00 -> 45.2 mm
- net Net-(D27-A): track 0.00 -> 40.7 mm
- net Net-(D26-A): track 0.00 -> 40.7 mm
- net Net-(D25-A): track 0.00 -> 40.7 mm
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
Commit message: routing
Parts:
- moved D82 35.0 mm to (330.2, 72.2)
- moved D78 30.9 mm to (296.0, 65.0)
- moved D72 22.9 mm to (288.3, 70.4)
- moved D75 22.9 mm to (326.4, 70.4)
- moved D77 19.0 mm to (303.6, 68.6)
- moved D14 16.8 mm to (315.0, 65.0)
- moved D81 12.0 mm to (299.8, 66.8)
- moved D79 8.41 mm to (322.6, 68.6)
- moved D83 8.41 mm to (307.4, 70.4)
- moved D76 4.21 mm to (311.2, 72.2)
Connections:
- D77 pad 2: unconnected-(D77-A-Pad2) -> Net-(D77-A)
- SW77 pad 2: unconnected-(SW77-Pad2) -> Net-(D77-A)
Routing:
- net row0: track 13.7 -> 274.2 mm
- net row4: track 0.00 -> 243.2 mm, vias 0 -> 1
- net row1: track 41.3 -> 282.6 mm
- net row3: track 0.00 -> 235.6 mm, vias 0 -> 2
- net row2: track 0.00 -> 212.5 mm, vias 0 -> 1
- net Net-(D81-A): track 0.00 -> 173.0 mm
- net Net-(D77-A): track 0.00 -> 161.9 mm
- net Net-(D78-A): track 0.00 -> 157.7 mm
- net Net-(D72-A): track 0.00 -> 142.4 mm
- net Net-(D76-A): track 0.00 -> 105.5 mm
- net Net-(D80-A): track 0.00 -> 102.1 mm
- net Net-(D79-A): track 0.00 -> 101.1 mm
- net Net-(D83-A): track 0.00 -> 94.1 mm
- net Net-(D75-A): track 0.00 -> 81.7 mm
- net Net-(D82-A): track 0.00 -> 58.6 mm
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
Commit message: update nets
Connections:
- A1 pad 5: col14 -> unconnected-(A1-GPIO3-Pad5)
- A1 pad 6: col14 -> col16
- A1 pad 7: col14 -> col15
- SW57 pad 1: col11 -> col13
- SW73 pad 1: col9 -> col10
- SW74 pad 1: col10 -> col11
- SW75 pad 1: col14 -> col15
- SW76 pad 1: col14 -> col15
- SW77 pad 1: col14 -> col15
- SW78 pad 1: col14 -> col15
- SW79 pad 1: col14 -> col16
- SW80 pad 1: col14 -> col16
- SW81 pad 1: col14 -> col16
Routing:
- net col16: track 0.00 -> 76.2 mm
- net col15: track 0.00 -> 76.2 mm
- net col14: track 0.00 -> 69.6 mm
- net col13: track 22.0 -> 87.4 mm
- net row1: track 282.6 -> 241.3 mm
- net col9: track 102.1 -> 67.0 mm
- net col10: track 113.1 -> 98.8 mm
- net row0: track 274.2 -> 260.5 mm
- net col12: track 63.8 -> 73.3 mm
- net col11: track 96.8 -> 106.3 mm
- net col6: track 87.0 -> 94.2 mm

Commit message: routing
Parts:
- added ?: , , F.Cu at (346.5, 81.5)
- added REF**: MountingHole_2.2mm_M2_Pad, MountingHole:MountingHole_2.2mm_M2_Pad, F.Cu at (304.4, 64.0)
Routing:
- net col0: track 88.8 -> 391.7 mm
- net col1: track 87.5 -> 366.1 mm
- net col2: track 89.0 -> 343.4 mm
- net col3: track 67.0 -> 317.4 mm
- net col4: track 67.0 -> 297.9 mm
- net col5: track 67.0 -> 282.4 mm
- net col6: track 94.2 -> 277.3 mm
- net col7: track 71.1 -> 244.3 mm
- net col8: track 67.0 -> 221.0 mm
- net col9: track 67.0 -> 201.8 mm
- net col10: track 98.8 -> 186.4 mm
- net col12: track 73.3 -> 133.1 mm
- net col11: track 106.3 -> 164.5 mm
- net col13: track 87.4 -> 119.8 mm
