File: discipline-pcb.kicad_pcb (KiCad board)
At the start: 2 copper layers, 357.2 x 120.3 mm, 219 parts, among them SW1 KEYSW, SW10 KEYSW, SW11 KEYSW, SW12 KEYSW, SW13 KEYSW, SW14 KEYSW, SW16 KEYSW, SW17 KEYSW, SW18 KEYSW, SW19 KEYSW, SW2 KEYSW, SW20 KEYSW, SW21 KEYSW, SW22 KEYSW, SW23 KEYSW, SW24 KEYSW, SW25 KEYSW, SW26 KEYSW, SW27 KEYSW, SW28 KEYSW, SW29 KEYSW, SW3 KEYSW, SW31 KEYSW, SW32 KEYSW, SW33 KEYSW, SW34 KEYSW, SW35 KEYSW, SW36 KEYSW, SW37 KEYSW, SW38 KEYSW, SW39 KEYSW, SW4 KEYSW, SW40 KEYSW, SW41 KEYSW, SW42 KEYSW, SW43 KEYSW, SW45 KEYSW, SW46 KEYSW, SW47 KEYSW, SW48 KEYSW, SW49 KEYSW, SW5 KEYSW, SW50 KEYSW, SW51 KEYSW, SW52 KEYSW, SW53 KEYSW, SW54 KEYSW, SW55 KEYSW, SW56 KEYSW, SW57 KEYSW, SW59 KEYSW, SW6 KEYSW, SW60 KEYSW, SW61 KEYSW, SW62 KEYSW, SW7 KEYSW, SW72 KEYSW, SW73 KEYSW, SW74 KEYSW, SW75 KEYSW, SW76 KEYSW, SW77 KEYSW, SW78 KEYSW, SW79 KEYSW, SW8 KEYSW, SW80 KEYSW, SW81 KEYSW, SW82 KEYSW, SW83 KEYSW, SW9 KEYSW, U1 SN74AHCT125N

Commit message: rotate led footprints
Parts:
- moved C13 4.00 mm to (397.5, 157.0)
- moved C14 4.00 mm to (397.5, 101.5)
- moved C10 3.00 mm to (217.4, 168.0)
- moved C11 3.00 mm to (286.3, 168.0)
- moved C12 3.00 mm to (346.6, 168.0)
- moved C8 3.00 mm to (77.7, 168.0)
- moved C9 3.00 mm to (144.4, 168.0)
- turned LED1 to 90 degrees
- turned LED10 to -90 degrees
- turned LED11 to -90 degrees
- turned LED12 to -90 degrees
- turned LED13 to 0 degrees
- turned LED14 to 0 degrees
- turned LED15 to 90 degrees
- turned LED2 to 90 degrees
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Connections:
- SW-RST1 pad 2: GND -> VSYS

Commit message: basic LED routing
Routing:
- net VSYS: track 0.00 -> 948.0 mm
- net Net-(LED12-DOUT): track 0.00 -> 83.8 mm
- net Net-(LED3-DOUT): track 0.00 -> 75.6 mm
- net Net-(LED10-DIN): track 0.00 -> 71.7 mm
- net Net-(LED10-DOUT): track 0.00 -> 68.9 mm
- net Net-(LED8-DOUT): track 0.00 -> 66.8 mm
- net Net-(LED7-DOUT): track 0.00 -> 61.5 mm
- net Net-(LED11-DOUT): track 0.00 -> 60.4 mm
- net Net-(LED2-DOUT): track 0.00 -> 57.4 mm
- net Net-(LED4-DOUT): track 0.00 -> 57.3 mm
- net Net-(LED5-DOUT): track 0.00 -> 57.0 mm
- net Net-(LED13-DOUT): track 0.00 -> 55.0 mm
- net Net-(LED1-DOUT): track 0.00 -> 54.5 mm
- net Net-(LED14-DOUT): track 0.00 -> 52.6 mm
- net Net-(LED6-DOUT): track 0.00 -> 34.1 mm

Commit message: at point of q's
Parts:
- moved D47 4.21 mm to (120.8, 72.2)
- moved D61 4.21 mm to (117.0, 70.4)
Connections:
- SW-RST1 pad 2: VSYS -> GND
Routing:
- net Net-(D62-A): track 0.00 -> 104.9 mm
- net Net-(D61-A): track 0.00 -> 103.5 mm
- net Net-(D60-A): track 0.00 -> 103.4 mm
- net Net-(D59-A): track 0.00 -> 100.8 mm
- net col2: track 0.00 -> 89.0 mm
- net col1: track 0.00 -> 85.1 mm
- net col0: track 0.00 -> 85.1 mm
- net Net-(D51-A): track 0.00 -> 82.4 mm
- net Net-(D50-A): track 0.00 -> 82.4 mm
- net Net-(D46-A): track 0.00 -> 81.9 mm
- net Net-(D47-A): track 0.00 -> 81.7 mm
- net Net-(D49-A): track 0.00 -> 81.6 mm
- net Net-(D48-A): track 0.00 -> 81.0 mm
- net Net-(D45-A): track 0.00 -> 76.6 mm
- net Net-(D38-A): track 0.00 -> 72.2 mm
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