File: base/base.kicad_pcb (KiCad board)
At the start: 2 copper layers, 366.2 x 134.3 mm, 6 parts

Commit message: update base to match holes in pcb
Parts:
- added ?: , , B.Cu at (85.4, 61.9)
- added ?: , , B.Cu at (276.6, 62.9)
- added ?: , , B.Cu at (269.4, 119.7)
- added ?: , , B.Cu at (191.9, 54.7)
- added ?: , , B.Cu at (375.1, 119.4)
- added ?: , , B.Cu at (61.1, 119.2)
- added ?: , , B.Cu at (145.4, 119.7)
- added ?: , , B.Cu at (369.7, 49.3)
Other:
- outline, holes or cut-outs redrawn
- rule pad_to_mask_clearance: 0 -> 0.051
- board text added: "kara70"
